Commit message: Refactored Gait and fixed forward.py coordinates

File: snakebot_ws/src/snakebot/urdf/snakebot.urdf (robot description, URDF)
Before this commit: robot snakebot, 22 links, 21 joints
Joints:
- joint rod_eight_joint: limit lower=-3.14 upper=3.14 effort=1000 velocity=0.1 -> lower=-3.14 upper=3.14 effort=1000 velocity=0.5
- joint rod_eleven_joint: limit lower=-3.14 upper=3.14 effort=1000 velocity=0.1 -> lower=-3.14 upper=3.14 effort=1000 velocity=0.5
- joint rod_five_joint: limit lower=-3.14 upper=3.14 effort=1000 velocity=0.1 -> lower=-3.14 upper=3.14 effort=1000 velocity=0.5
- joint rod_four_joint: limit lower=-3.14 upper=3.14 effort=1000 velocity=0.1 -> lower=-3.14 upper=3.14 effort=1000 velocity=0.5
- joint rod_nine_joint: limit lower=-3.14 upper=3.14 effort=1000 velocity=0.1 -> lower=-3.14 upper=3.14 effort=1000 velocity=0.5
- joint rod_one_joint: limit lower=-3.14 upper=3.14 effort=1000 velocity=0.1 -> lower=-3.14 upper=3.14 effort=1000 velocity=0.5
- joint rod_seven_joint: limit lower=-3.14 upper=3.14 effort=1000 velocity=0.1 -> lower=-3.14 upper=3.14 effort=1000 velocity=0.5
- joint rod_six_joint: limit lower=-3.14 upper=3.14 effort=1000 velocity=0.1 -> lower=-3.14 upper=3.14 effort=1000 velocity=0.5
- joint rod_ten_joint: limit lower=-3.14 upper=3.14 effort=1000 velocity=0.1 -> lower=-3.14 upper=3.14 effort=1000 velocity=0.5
- joint rod_three_joint: limit lower=-3.14 upper=3.14 effort=1000 velocity=0.1 -> lower=-3.14 upper=3.14 effort=1000 velocity=0.5
