Commit message: Added LIDAR scanner; needs objects

File: snakebot_ws/src/snakebot/urdf/snakebot.xacro (robot description, xacro)
@@ -43,3 +43,56 @@
         </plugin>
     </gazebo>
+    <link name="lidar_link">
+        <inertial>
+            <mass value="0.1"/>
+            <origin xyz="0 0 0" rpy="0 0 0"/>
+            <inertia ixx="1e-5" ixy="0.0" ixz="0.0" iyy="1e-5" iyz="0.0" izz="1e-5"/>
+        </inertial>
+        <visual>
+            <geometry>
+                <cylinder radius="0.05" length="0.1"/>
+            </geometry>
+            <origin xyz="0 0 0.05" rpy="0 0 0"/>
+            <material name="gray">
+                <color rgba="0.5 0.5 0.5 1.0"/>
+            </material>
+        </visual>
+        <collision>
+            <geometry>
+                <cylinder radius="0.05" length="0.1"/>
+            </geometry>
+            <origin xyz="0 0 0.05" rpy="0 0 0"/>
+        </collision>
+    </link>
+    <joint name="lidar_joint" type="fixed">
+        <parent link="base_link"/>
+        <child link="lidar_link"/>
+        <origin xyz="0 0 0.1" rpy="0 0 0"/>
+    </joint>
+    <gazebo reference="lidar_link">
+        <sensor name="lidar" type="gpu_lidar">
+            <always_on>true</always_on>
+            <update_rate>10</update_rate>
+            <visualize>true</visualize>
+            <ray>
+                <scan>
+                    <horizontal>
+                        <samples>720</samples>
+                        <resolution>1</resolution>
+                        <min_angle>-1.5708</min_angle>
+                        <max_angle>1.5708</max_angle>
+                    </horizontal>
+                </scan>
+                <range>
+                    <min>0.1</min>
+                    <max>10.0</max>
+                    <resolution>0.01</resolution>
+                </range>
+            </ray>
+            <plugin name="gazebo_ros_laser_controller" filename="libgazebo_ros_gpu_laser.so">
+                <topicName>/scan</topicName>
+                <frameName>lidar_link</frameName>
+            </plugin>
+        </sensor>
+    </gazebo>
 </robot>

Commit message: added rear lidar

File: snakebot_ws/src/snakebot/urdf/snakebot.xacro (robot description, xacro)
@@ -43,4 +43,5 @@
         </plugin>
     </gazebo>
+    <!-- Front LIDAR -->
     <link name="lidar_link">
         <inertial>
@@ -96,3 +97,57 @@
         </sensor>
     </gazebo>
+    <!-- Rear LIDAR -->
+    <link name="rear_lidar_link">
+        <inertial>
+            <mass value="0.1"/>
+            <origin xyz="0 0 0" rpy="0 0 0"/>
+            <inertia ixx="1e-5" ixy="0.0" ixz="0.0" iyy="1e-5" iyz="0.0" izz="1e-5"/>
+        </inertial>
+        <visual>
+            <geometry>
+                <cylinder radius="0.05" length="0.1"/>
+            </geometry>
+            <origin xyz="0 0 0.05" rpy="0 0 0"/>
+            <material name="gray">
+                <color rgba="0.5 0.5 0.5 1.0"/>
+            </material>
+        </visual>
+        <collision>
+            <geometry>
+                <cylinder radius="0.05" length="0.1"/>
+            </geometry>
+            <origin xyz="0 0 0.05" rpy="0 0 0"/>
+        </collision>
+    </link>
+    <joint name="rear_lidar_joint" type="fixed">
+        <parent link="rod_eleven"/>
+        <child link="rear_lidar_link"/>
+        <origin xyz="0 0 0.1" rpy="0 0 0"/>
+    </joint>
+    <gazebo reference="rear_lidar_link">
+        <sensor name="rear_lidar" type="gpu_lidar">
+            <always_on>true</always_on>
+            <update_rate>10</update_rate>
+            <visualize>true</visualize>
+            <ray>
+                <scan>
+                    <horizontal>
+                        <samples>720</samples>
+                        <resolution>1</resolution>
+                        <min_angle>-1.5708</min_angle>
+                        <max_angle>1.5708</max_angle>
+                    </horizontal>
+                </scan>
+                <range>
+                    <min>0.1</min>
+                    <max>10.0</max>
+                    <resolution>0.01</resolution>
+                </range>
+            </ray>
+            <plugin name="gazebo_ros_rear_laser_controller" filename="libgazebo_ros_gpu_laser.so">
+                <topicName>/rear_scan</topicName>
+                <frameName>rear_lidar_link</frameName>
+            </plugin>
+        </sensor>
+    </gazebo>
 </robot>

Commit message: Added vizualization to Lidar

File: snakebot_ws/src/snakebot/urdf/snakebot.xacro (robot description, xacro)
@@ -69,39 +69,28 @@
         <parent link="base_link"/>
         <child link="lidar_link"/>
-        <origin xyz="0 0 0.1" rpy="0 0 0"/>
+        <origin xyz="0 0 0.1" rpy="0 0 3.14159"/>
     </joint>
     <gazebo reference="lidar_link">
-        <sensor name="lidar" type="gpu_lidar">
-            <always_on>true</always_on>
+        <sensor name="lidar" type="ray">
+            <visualize>true</visualize>
             <update_rate>10</update_rate>
-            <visualize>true</visualize>
             <ray>
                 <scan>
-                    <horizontal>
-                        <samples>720</samples>
-                        <resolution>1</resolution>
-                        <min_angle>-1.5708</min_angle>
-                        <max_angle>1.5708</max_angle>
-                    </horizontal>
+                <horizontal>
+                    <samples>100</samples>
+                    <min_angle>-1.05</min_angle>
+                    <max_angle>1.05</max_angle>
+                </horizontal>
                 </scan>
                 <range>
-                    <min>0.1</min>
-                    <max>10.0</max>
-                    <resolution>0.01</resolution>
+                    <min>0.3</min>
+                    <max>10</max>
                 </range>
             </ray>
-            <plugin name="gazebo_ros_laser_controller" filename="libgazebo_ros_gpu_laser.so">
-                <topicName>/scan</topicName>
-                <frameName>lidar_link</frameName>
-            </plugin>
+            <plugin filename="VisualizeLidar" name="Visualize Lidar"></plugin>
         </sensor>
     </gazebo>
     <!-- Rear LIDAR -->
     <link name="rear_lidar_link">
-        <inertial>
-            <mass value="0.1"/>
-            <origin xyz="0 0 0" rpy="0 0 0"/>
-            <inertia ixx="1e-5" ixy="0.0" ixz="0.0" iyy="1e-5" iyz="0.0" izz="1e-5"/>
-        </inertial>
         <visual>
             <geometry>
@@ -110,44 +99,86 @@
             <origin xyz="0 0 0.05" rpy="0 0 0"/>
             <material name="gray">
-                <color rgba="0.5 0.5 0.5 1.0"/>
+                <color rgba="0.4 0.4 0.4 1.0"/>
             </material>
         </visual>
-        <collision>
-            <geometry>
-                <cylinder radius="0.05" length="0.1"/>
-            </geometry>
-            <origin xyz="0 0 0.05" rpy="0 0 0"/>
-        </collision>
     </link>
     <joint name="rear_lidar_joint" type="fixed">
-        <parent link="rod_eleven"/>
+        <parent link="link_ten"/>
         <child link="rear_lidar_link"/>
         <origin xyz="0 0 0.1" rpy="0 0 0"/>
     </joint>
     <gazebo reference="rear_lidar_link">
-        <sensor name="rear_lidar" type="gpu_lidar">
-            <always_on>true</always_on>
+        <sensor name="rear_lidar" type="ray">
+            <visualize>true</visualize>
             <update_rate>10</update_rate>
-            <visualize>true</visualize>
             <ray>
                 <scan>
                     <horizontal>
-                        <samples>720</samples>
-                        <resolution>1</resolution>
-                        <min_angle>-1.5708</min_angle>
-                        <max_angle>1.5708</max_angle>
+                        <samples>100</samples>
+                        <min_angle>-1.0</min_angle>
+                        <max_angle>1.0</max_angle>
                     </horizontal>
                 </scan>
                 <range>
-                    <min>0.1</min>
-                    <max>10.0</max>
-                    <resolution>0.01</resolution>
+                    <min>0.3</min>
+                    <max>5</max>
                 </range>
             </ray>
-            <plugin name="gazebo_ros_rear_laser_controller" filename="libgazebo_ros_gpu_laser.so">
-                <topicName>/rear_scan</topicName>
-                <frameName>rear_lidar_link</frameName>
+            <plugin name="rear_lidar_plugin" filename="libgazebo_ros_ray_sensor.so">
+                <ros>
+                    <argument>~/out:=rear_scan</argument>
+                </ros>
+                <output_type>sensor_msgs/LaserScan</output_type>
+                <frame_name>rear_laser_frame</frame_name>
             </plugin>
         </sensor>
     </gazebo>
+    <!-- Side IR Sensor Macro -->
+    <xacro:macro name="side_ir_sensor" params="sensor_id parent_link topic_name">
+        <link name="${sensor_id}_link">
+            <visual>
+                <geometry>
+                    <box size="0.02 0.02 0.02"/>
+                </geometry>
+                <origin xyz="0 0 0" rpy="0 0 0"/>
+                <material name="blue">
+                    <color rgba="0.2 0.2 1.0 1.0"/>
+                </material>
+            </visual>
+        </link>
+        <joint name="${sensor_id}_joint" type="fixed">
+            <parent link="${parent_link}"/>
+            <child link="${sensor_id}_link"/>
+            <origin xyz="0.05 0 0" rpy="0 0 0"/>
+        </joint>
+        <gazebo reference="${sensor_id}_link">
+            <sensor name="${sensor_id}" type="ray">
+                <update_rate>10</update_rate>
+                <ray>
+                    <scan>
+                        <horizontal>
+                            <samples>20</samples>
+                            <min_angle>-0.35</min_angle>
+                            <max_angle>0.35</max_angle>
+                        </horizontal>
+                    </scan>
+                    <range>
+                        <min>0.05</min>
+                        <max>0.5</max>
+                    </range>
+                </ray>
+                <plugin name="${sensor_id}_plugin" filename="libgazebo_ros_ray_sensor.so">
+                    <ros>
+                        <argument>~/out:=${topic_name}</argument>
+                    </ros>
+                    <output_type>sensor_msgs/LaserScan</output_type>
+                    <frame_name>${sensor_id}_frame</frame_name>
+                </plugin>
+            </sensor>
+        </gazebo>
+    </xacro:macro>
+    <!-- Side IR sensors on links 4, 6, 8 -->
+    <xacro:side_ir_sensor sensor_id="ir_link4" parent_link="link_four" topic_name="ir_link4_scan"/>
+    <xacro:side_ir_sensor sensor_id="ir_link6" parent_link="link_six" topic_name="ir_link6_scan"/>
+    <xacro:side_ir_sensor sensor_id="ir_link8" parent_link="link_eight" topic_name="ir_link8_scan"/>
 </robot>
